Commit message: Update solution

File: HW05/Solution/Tinker Twins/3RRR/URDF/3RRR/urdf/3RRR.urdf (robot description, URDF)
Before this commit: robot 3RRR, 13 links, 12 joints
Links:
- link Base: mass 1.0550351703688 -> 0.97649535402911
- link Distal_Link_3: mass 0.10961899508206 -> 0.109618995082061
- link Platform_1: mass 0.204748162200487 -> 0.204748162200477
- link Platform_2: mass 0.204748162200487 -> 0.204748162200477
- link Platform_3: mass 0.204748162200487 -> 0.204748162200477
- link Proximal_Link_1: mass 0.124327488543994 -> 0.124327488543993
- link Proximal_Link_2: mass 0.124327488543994 -> 0.124327488543995
- link Proximal_Link_3: mass 0.124327488543995 -> 0.124327488543994
Joints:
- joint Distal_Joint_1: origin xyz=-0.000932984996129982 0.299998549228158 0.00999999999999995 rpy=0 0 0 -> xyz=-0.0244720942079539 0.299000194991704 0.00999999999999996 rpy=0 0 0
- joint Distal_Joint_2: origin xyz=-0.289175787686616 -0.0798583575428643 0.00999999999999994 rpy=0 0 0 -> xyz=-0.271689174071722 -0.127220252681032 0.00999999999999996 rpy=0 0 0
- joint Distal_Joint_3: origin xyz=0.298599347923383 -0.0289557149727769 0.0100000000000005 rpy=0 0 0 -> xyz=0.299970063562069 0.00423803805647649 0.0100000000000003 rpy=0 0 0
- joint Pen_Joint_1: origin xyz=0.0866025100946133 -0.0499999825156222 -0.0499999999999999 rpy=0 0 0 -> xyz=0.0866025100946145 -0.0499999825156214 -0.0499999999999999 rpy=0 0 0
- joint Pen_Joint_2: origin xyz=0 0.099999965031245 -0.0500000000000001 rpy=0 0 0 -> xyz=0 0.0999999650312451 -0.0500000000000001 rpy=0 0 0
- joint Pen_Joint_3: origin xyz=-0.086602510094613 -0.0499999825156237 -0.05 rpy=0 0 0 -> xyz=-0.0866025100946132 -0.0499999825156224 -0.0500000000000001 rpy=0 0 0
- joint Platform_Joint_1: origin xyz=0.245788708401739 -0.0224985492281455 0.0100000000000001 rpy=0 0 0 -> xyz=0.247677182518953 -0.0340001949916939 0.00999999999999986 rpy=0 0 0
- joint Platform_Joint_2: origin xyz=0.0577175189590905 0.207358413931771 0.0100000000000002 rpy=0 0 0 -> xyz=0.0618815302066741 0.242220305134155 0.01 rpy=0 0 0
- joint Platform_Joint_3: origin xyz=-0.161996851988848 -0.181044265896015 0.00999999999999979 rpy=0 0 0 -> xyz=-0.163367576197156 -0.189238038056475 0.00999999999999971 rpy=0 0 0
- joint Proximal_Joint_1: origin xyz=-0.281458256229922 -0.162500000000012 0.03 rpy=0 0 0 -> xyz=-0.259807621135314 -0.15000000000001 0.03 rpy=0 0 0
- joint Proximal_Joint_2: origin xyz=0.281458245997827 -0.162500003935774 0.03 rpy=0 0 0 -> xyz=0.259807621135349 -0.14999999999999 0.03 rpy=0 0 0
- joint Proximal_Joint_3: origin xyz=0 0.324999980868794 0.0299999999999999 rpy=0 0 0 -> xyz=0 0.3 0.03 rpy=0 0 0
